File: pcb/EAGLE/projects/3YP PCB/schematic.sch (EAGLE design)
At the start: 29 parts, among them IC1 ATSAMR30M18A-I_RM100, IC2 TLS850B0TBV33ATMA1, IC3 DS18B20U+, J1 19-46-1-TGG, U1 1042P

Commit message: Added parts list and amlost finished with schematic
Parts:
- removed C3: 1u, rcl:C-EUC0805
- added C6: 1u, rcl:C-EUC0805
- added C7: 100n, rcl:C-EUC0805
- C4: value 100n -> 1u
- C5: value 100u -> 100n; device rcl:CPOL-EUA/3216-18W -> rcl:C-EUC0805
- IC2: value TLS850B0TBV33ATMA1 -> LD39015M33R; device SamacSys_Parts:TLS850B0TBV33ATMA1 -> SamacSys_Parts:LD39015M33R
- L1: device rcl:L-EUL0201 -> SamacSys_Parts:MHQ1005P10NJT
- S1, S2: value 4-1437565-1 -> PTS645SM43SMTR92LFS; device SamacSys_Parts:4-1437565-1 -> SamacSys_Parts:PTS645SM43SMTR92LFS
- S3: value MIC94163YCS-TR -> SIP32431DR3-T1GE3; device SamacSys_Parts:MIC94163YCS-TR -> SamacSys_Parts:SIP32431DR3-T1GE3
- SV1: value (none) -> M20-9980445; device con-lstb:MA04-2 -> SamacSys_Parts:M20-9980445
Connections:
- net BATTERY_IN: now also IC2.IN; no longer C5.+, IC2.I
- net DS18_POW: now also C7.1, S3.OUT; no longer S3.VOUT_1, S3.VOUT_2
- net GND: now also C5.2, C6.2, C7.2, S1.4, S2.4, S3.GND_1, S3.GND_2; no longer C3.2, C5.-, IC2.TAB, S1.1, S2.1, S3.GND
- net N$1: now also S2.1; no longer S2.4
- net N$8: now also S1.1; no longer S1.4
- net PA19_DS18_EN: now also S3.ON/OFF; no longer S3.EN
- net VCC: now also C5.1, C6.1, IC2.OUT, S3.IN; no longer C3.1, IC2.Q, S3.VIN_1, S3.VIN_2
Other:
- moved on the sheet: C4, J1, S3, SV1, U1
