File: pcb/EAGLE/projects/3YP PCB Rev2A/3yp_node.brd (EAGLE design)
At the start: 105.4 x 29.8 mm, 32 parts, among them IC1 ATSAMR30M18A-I_RM100, IC2 LD39015M33R, IC3 DS18B20U+, IC4 AT25DF321A-SH-B, J1 19-46-1-TGG, J2 TSW-104-07-F-S, U1 1042P

Commit message: Updated board
Parts:
- moved U1 0.64 mm to (46.4, 13.6)
- moved R12 0.25 mm to (94.6, 23.9)
Routing:
- net N$10: track 24.8 -> 23.4 mm
- net VCC: track 131.4 -> 132.6 mm
- net PA09_I2C_SCL: track 69.9 -> 71.1 mm
- net PA08_I2C_SDA: track 50.7 -> 51.4 mm

Commit message: Not too sure what has changed, but am sure something has
Parts:
- added C7: 100n, rcl:C0805
- added HM1: SI7006-A20-IM1, SamacSys_Parts:SON100P300X300X80-7N
Connections:
- net DS18_POW: now also C7.1, HM1.5
- net GND: now also C7.2, HM1.2
- net PA08_I2C_SDA: now also HM1.1
- net PA09_I2C_SCL: now also HM1.6
Routing:
- net PA09_I2C_SCL: track 71.1 -> 94.9 mm
- net PA08_I2C_SDA: track 51.4 -> 70.7 mm
- net DS18_POW: track 6.87 -> 22.1 mm, vias 0 -> 2
- net NRESET: track 54.8 -> 54.9 mm, vias 0 -> 2
Other:
- board text added: "REV 2B MARCH 2020 SAMUEL KENDALL UNI OF SOUTHAMPTON"
- board text removed: "REV 2A MARCH 2020 SAMUEL KENDALL UNI OF SOUTHAMPTON"

Commit message: Finalising board...
Parts:
- C1: value 100u -> 10u; device rcl:A/3216-18W -> SamacSys_Parts:CAPPM2014X170N
- C4: value 100n -> 1u
- moved C5 30.6 mm to (65.7, 15.1)
- moved C1 0.77 mm to (65.7, 19.4), turned to 90 degrees
Connections:
- net GND: now also C1.2; no longer C1.-
- net VCC: now also C1.1; no longer C1.+
Routing:
- net VCC: track 132.6 -> 134.8 mm
