File: pcb/EAGLE/projects/3YP PCB Rev2A/3yp_node.brd (EAGLE design)
At the start: 105.4 x 29.8 mm, 34 parts, among them IC1 ATSAMR30M18A-I_RM100, IC2 LD39015M33R, IC3 DS18B20U+, IC4 AT25DF321A-SH-B, J1 19-46-1-TGG, J2 TSW-104-07-F-S, U1 1042P

Commit message: Regenned files
Parts:
- added C10, C9: 100n, rcl:C0805
- added C8: 10u, SamacSys_Parts:CAPPM2014X170N
- moved C6 3.02 mm to (58.5, 20.2), turned to 180 degrees
- moved C1 2.22 mm to (63.8, 20.6)
- moved R1 1.40 mm to (73.9, 27.7), turned to 270 degrees
Connections:
- net GND: now also C10.1, C8.2, C9.2
- net VCC: now also C10.2, C8.1, C9.1
Routing:
- net VCC: track 134.8 -> 137.0 mm
- net !PA15_SPI_FLASH_SS: track 33.2 -> 31.3 mm
- net PA19_SPI_SCK: track 44.1 -> 42.5 mm
- net DS18_POW: track 22.1 -> 22.9 mm
- net !PA06_SPI_FLASH_HOLD: track 33.7 -> 33.0 mm
- net PA27_DS18_DQ: track 6.19 -> 5.50 mm
- net N$2: track 4.53 -> 3.86 mm
