File: pcb/EAGLE/projects/3YP PCB Rev2A/3yp_node.sch (EAGLE design)
At the start: 32 parts, among them IC1 ATSAMR30M18A-I_RM100, IC2 LD39015M33R, IC3 DS18B20U+, IC4 AT25DF321A-SH-B, J1 19-46-1-TGG, J2 TSW-104-07-F-S, U1 1042P

Commit message: Updated board
Connections:
- net VCC: now also IC2.VCC; no longer IC2.OUT
Changed lines of the file:
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@@
 <pinref part="C4" gate="G$1" pin="1"/>
 <wire x1="226.06" y1="152.4" x2="226.06" y2="149.86" width="0.1524" layer="91"/>
-<pinref part="IC2" gate="G$1" pin="OUT"/>
+<pinref part="IC2" gate="G$1" pin="VCC"/>
 <wire x1="223.52" y1="152.4" x2="226.06" y2="152.4" width="0.1524" layer="91"/>
 <junction x="226.06" y="152.4"/>
@@
 </sheet>
 </sheets>
+<errors>
+</errors>
 </schematic>
 </drawing>

Commit message: Not too sure what has changed, but am sure something has
Parts:
- added C7: 100n, rcl:C-EUC0805
- added HM1: SI7006-A20-IM1, SamacSys_Parts:SI7006-A20-IM1
Connections:
- net DS18_POW: now also C7.1, HM1.VCC
- net GND: now also C7.2, HM1.GND
- net PA08_I2C_SDA: now also HM1.SDA
- net PA09_I2C_SCL: now also HM1.SCL
Other:
- moved on the sheet: C3, C4, IC2, U1

Commit message: Finalising board...
Parts:
- C1: value 100u -> 10u; device rcl:CPOL-EUA/3216-18W -> SamacSys_Parts:TAJP106K006RNJ
- C4: value 100n -> 1u
Changed lines of the file:
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@@
 <part name="R5" library="rcl" library_urn="urn:adsk.eagle:library:334" deviceset="R-EU_" device="R0603" package3d_urn="urn:adsk.eagle:package:23555/3" value="100"/>
 <part name="R6" library="rcl" library_urn="urn:adsk.eagle:library:334" deviceset="R-EU_" device="R0603" package3d_urn="urn:adsk.eagle:package:23555/3" value="100"/>
-<part name="C1" library="rcl" library_urn="urn:adsk.eagle:library:334" deviceset="CPOL-EU" device="A/3216-18W" package3d_urn="urn:adsk.eagle:package:23408/2" value="100u"/>
+<part name="C1" library="SamacSys_Parts" deviceset="TAJP106K006RNJ" device="" value="10u"/>
 <part name="P+2" library="supply1" library_urn="urn:adsk.eagle:library:371" deviceset="VCC" device=""/>
 <part name="GND5" library="supply1" library_urn="urn:adsk.eagle:library:371" deviceset="GND" device=""/>
@@
 <part name="IC2" library="SamacSys_Parts" deviceset="LD39015M33R" device=""/>
 <part name="C3" library="rcl" library_urn="urn:adsk.eagle:library:334" deviceset="C-EU" device="C0805" package3d_urn="urn:adsk.eagle:package:23617/2" value="1u"/>
-<part name="C4" library="rcl" library_urn="urn:adsk.eagle:library:334" deviceset="C-EU" device="C0805" package3d_urn="urn:adsk.eagle:package:23617/2" value="100n"/>
+<part name="C4" library="rcl" library_urn="urn:adsk.eagle:library:334" deviceset="C-EU" device="C0805" package3d_urn="urn:adsk.eagle:package:23617/2" value="1u"/>
 <part name="J2" library="SamacSys_Parts" deviceset="TSW-104-07-F-S" device=""/>
 <part name="IC4" library="SamacSys_Parts" deviceset="AT25DF321A-SH-B" device=""/>
@@
 <attribute name="VALUE" x="81.28" y="99.06" size="1.778" layer="96" rot="R180"/>
 </instance>
-<instance part="GND1" gate="1" x="83.82" y="86.36" smashed="yes">
-<attribute name="VALUE" x="81.28" y="83.82" size="1.778" layer="96"/>
+<instance part="GND1" gate="1" x="83.82" y="81.28" smashed="yes">
+<attribute name="VALUE" x="81.28" y="78.74" size="1.778" layer="96"/>
 </instance>
 <instance part="IC1" gate="G$1" x="144.78" y="99.06" smashed="yes" rot="R180">
@@
 <attribute name="VALUE" x="127.762" y="77.47" size="1.778" layer="96" rot="R90"/>
 </instance>
-<instance part="C1" gate="G$1" x="88.9" y="93.98" smashed="yes">
-<attribute name="NAME" x="90.424" y="94.361" size="1.778" layer="95"/>
-<attribute name="VALUE" x="90.424" y="89.281" size="1.778" layer="96"/>
+<instance part="C1" gate="G$1" x="88.9" y="96.52" smashed="yes" rot="R270">
+<attribute name="NAME" x="91.821" y="94.996" size="1.778" layer="95" rot="R270"/>
+<attribute name="VALUE" x="84.201" y="94.996" size="1.778" layer="96" rot="R270"/>
 </instance>
 <instance part="P+2" gate="VCC" x="35.56" y="127" smashed="yes">
@@
 <segment>
 <pinref part="GND1" gate="1" pin="GND"/>
-<wire x1="83.82" y1="88.9" x2="88.9" y2="88.9" width="0.1524" layer="91"/>
+<wire x1="83.82" y1="83.82" x2="88.9" y2="83.82" width="0.1524" layer="91"/>
 <pinref part="C1" gate="G$1" pin="-"/>
-<wire x1="88.9" y1="88.9" x2="109.22" y2="88.9" width="0.1524" layer="91"/>
-<junction x="88.9" y="88.9"/>
+<wire x1="88.9" y1="83.82" x2="109.22" y2="83.82" width="0.1524" layer="91"/>
+<junction x="88.9" y="83.82"/>
 <pinref part="IC1" gate="G$1" pin="GND_2"/>
-<wire x1="109.22" y1="99.06" x2="109.22" y2="88.9" width="0.1524" layer="91"/>
-</segment>
-<segment>
+<wire x1="109.22" y1="99.06" x2="109.22" y2="83.82" width="0.1524" layer="91"/>
+</segment>
+<segment>
