File: pcb/EAGLE/projects/3YP PCB Rev2A/3yp_node.sch (EAGLE design)
At the start: 34 parts, among them IC1 ATSAMR30M18A-I_RM100, IC2 LD39015M33R, IC3 DS18B20U+, IC4 AT25DF321A-SH-B, J1 19-46-1-TGG, J2 TSW-104-07-F-S, U1 1042P

Commit message: Regenned files
Parts:
- added C10, C9: 100n, rcl:C-EUC0805
- added C8: 10u, SamacSys_Parts:TAJP106K006RNJ
Connections:
- net GND: now also C10.1, C8.-, C9.2
- net VCC: now also C10.2, C8.+, C9.1
Changed lines of the file:
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@@
 <part name="C7" library="rcl" library_urn="urn:adsk.eagle:library:334" deviceset="C-EU" device="C0805" package3d_urn="urn:adsk.eagle:package:23617/2" value="100n"/>
 <part name="GND14" library="supply1" library_urn="urn:adsk.eagle:library:371" deviceset="GND" device=""/>
+<part name="C8" library="SamacSys_Parts" deviceset="TAJP106K006RNJ" device="" value="10u"/>
+<part name="GND19" library="supply1" library_urn="urn:adsk.eagle:library:371" deviceset="GND" device=""/>
+<part name="C9" library="rcl" library_urn="urn:adsk.eagle:library:334" deviceset="C-EU" device="C0805" package3d_urn="urn:adsk.eagle:package:23617/2" value="100n"/>
+<part name="C10" library="rcl" library_urn="urn:adsk.eagle:library:334" deviceset="C-EU" device="C0805" package3d_urn="urn:adsk.eagle:package:23617/2" value="100n"/>
 </parts>
 <sheets>
@@
 <text x="83.82" y="177.8" size="1.778" layer="91">RF Antenna Connector</text>
 <text x="213.36" y="180.34" size="1.778" layer="91">Battery Holder</text>
-<text x="55.88" y="33.02" size="1.778" layer="91">SPI Flash with Hold and no Write Protect (internal pull-up)</text>
+<text x="40.64" y="33.02" size="1.778" layer="91">SPI Flash with Hold and no Write Protect (internal pull-up)</text>
 </plain>
 <instances>
@@
 <attribute name="VALUE" x="220.98" y="106.68" size="1.778" layer="96"/>
 </instance>
+<instance part="C8" gate="G$1" x="104.14" y="22.86" smashed="yes">
+<attribute name="NAME" x="105.664" y="25.781" size="1.778" layer="95"/>
+<attribute name="VALUE" x="105.664" y="18.161" size="1.778" layer="96"/>
+</instance>
+<instance part="GND19" gate="1" x="121.92" y="22.86" smashed="yes" rot="R90">
+<attribute name="VALUE" x="124.46" y="20.32" size="1.778" layer="96" rot="R90"/>
+</instance>
+<instance part="C9" gate="G$1" x="109.22" y="30.48" smashed="yes" rot="R90">
+<attribute name="NAME" x="108.839" y="32.004" size="1.778" layer="95" rot="R90"/>
+<attribute name="VALUE" x="113.919" y="32.004" size="1.778" layer="96" rot="R90"/>
+</instance>
+<instance part="C10" gate="G$1" x="99.06" y="88.9" smashed="yes" rot="R180">
+<attribute name="NAME" x="105.156" y="88.519" size="1.778" layer="95" rot="R180"/>
+<attribute name="VALUE" x="105.156" y="93.599" size="1.778" layer="96" rot="R180"/>
+</instance>
 </instances>
 <busses>
@@
 <wire x1="83.82" y1="96.52" x2="88.9" y2="96.52" width="0.1524" layer="91"/>
 <pinref part="C1" gate="G$1" pin="+"/>
-<wire x1="88.9" y1="96.52" x2="106.68" y2="96.52" width="0.1524" layer="91"/>
+<wire x1="88.9" y1="96.52" x2="99.06" y2="96.52" width="0.1524" layer="91"/>
 <junction x="88.9" y="96.52"/>
+<wire x1="99.06" y1="96.52" x2="106.68" y2="96.52" width="0.1524" layer="91"/>
 <wire x1="106.68" y1="96.52" x2="106.68" y2="101.6" width="0.1524" layer="91"/>
 <pinref part="IC1" gate="G$1" pin="VDD"/>
 <wire x1="106.68" y1="101.6" x2="109.22" y2="101.6" width="0.1524" layer="91"/>
+<pinref part="C10" gate="G$1" pin="2"/>
+<wire x1="99.06" y1="93.98" x2="99.06" y2="96.52" width="0.1524" layer="91"/>
+<junction x="99.06" y="96.52"/>
 </segment>
 <segment>
@@
 <pinref part="P+9" gate="VCC" pin="VCC"/>
 <wire x1="101.6" y1="20.32" x2="101.6" y2="22.86" width="0.1524" layer="91"/>
+<pinref part="C8" gate="G$1" pin="+"/>
+<wire x1="104.14" y1="22.86" x2="101.6" y2="22.86" width="0.1524" layer="91"/>
+<junction x="101.6" y="22.86"/>
+<wire x1="104.14" y1="22.86" x2="104.14" y2="30.48" width="0.1524" layer="91"/>
+<junction x="104.14" y="22.86"/>
+<pinref part="C9" gate="G$1" pin="1"/>
+<wire x1="104.14" y1="30.48" x2="106.68" y2="30.48" width="0.1524" layer="91"/>
 </segment>
 </net>
@@
 <wire x1="83.82" y1="83.82" x2="88.9" y2="83.82" width="0.1524" layer="91"/>
 <pinref part="C1" gate="G$1" pin="-"/>
-<wire x1="88.9" y1="83.82" x2="109.22" y2="83.82" width="0.1524" layer="91"/>
+<wire x1="88.9" y1="83.82" x2="99.06" y2="83.82" width="0.1524" layer="91"/>
 <junction x="88.9" y="83.82"/>
 <pinref part="IC1" gate="G$1" pin="GND_2"/>
+<wire x1="99.06" y1="83.82" x2="109.22" y2="83.82" width="0.1524" layer="91"/>
 <wire x1="109.22" y1="99.06" x2="109.22" y2="83.82" width="0.1524" layer="91"/>
+<pinref part="C10" gate="G$1" pin="1"/>
+<wire x1="99.06" y1="86.36" x2="99.06" y2="83.82" width="0.1524" layer="91"/>
+<junction x="99.06" y="83.82"/>
 </segment>
 <segment>
@@
 <wire x1="223.52" y1="111.76" x2="223.52" y2="114.3" width="0.1524" layer="91"/>
 </segment>
+<segment>
+<pinref part="C8" gate="G$1" pin="-"/>
+<pinref part="GND19" gate="1" pin="GND"/>
+<wire x1="116.84" y1="22.86" x2="119.38" y2="22.86" width="0.1524" layer="91"/>
+<pinref part="C9" gate="G$1" pin="2"/>
+<wire x1="114.3" y1="30.48" x2="119.38" y2="30.48" width="0.1524" layer="91"/>
+<wire x1="119.38" y1="30.48" x2="119.38" y2="22.86" width="0.1524" layer="91"/>
+<junction x="119.38" y="22.86"/>
+</segment>
 </net>
