File: pcb/EAGLE/projects/Programmer/programmer_pcb2.sch (EAGLE design)
At the start: 53 parts, among them IC1 FT232HL-REEL, IC2 TPS78233DDCT, IC3 93LC56BT-E_OT, IC4 SN74LVC08ADRG4, IC5 NC7SZ04P5X, J1 MC-254-08-00-ST-DIP, J2 0480372200, J3 M20-9980545, J4 M20-9980545, Y1 9C-12.000MAAJ-T

Commit message: Assorted updates...
Other:
- note added: "12MHz Crystal"
- note added: "AND Gates to switch signals"
- note added: "Capacitors for line stability"
- note added: "EEPROM to store configuration#"
- note added: "Headers to expose IC pins"
- note added: "Inverter to provide !SWD"
- note added: "LEDs for RX and TX"
- note added: "Programming Header and Board Power Switch"
- note added: "Reset Switch"
- note added: "Resistors to power lines from USB"
- note added: "USB Connector"
- note added: "Voltage Regulator for MCU Power"
- moved on the sheet: C14, C18, IC5, J1, R5, S1, S3
